File: Interface-Tester/Interface-Tester.kicad_pcb (KiCad board)
At the start: 2 copper layers, 62.8 x 18.5 mm, 17 parts, among them J1 INTERFACE, J2 I2C, J3 PWR, SW1 SW, SW2 SW, SW3 SW, SW4 SW, SW5 SW, SW6 SW, SW7 SW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

Commit message: Version 1.1.0 of interface tester.
Parts:
- D1, D2, D3, D4, D5, D6: footprint Diodes_SMD:D_0603 -> LED_SMD:LED_0603_1608Metric
- J1: footprint Pin_Headers:Pin_Header_Straight_1x08_Pitch2.54mm -> Connector_PinHeader_2.54mm:PinHeader_1x08_P2.54mm_Vertical
- J2: footprint Pin_Headers:Pin_Header_Straight_1x04_Pitch2.54mm -> Connector_PinHeader_2.54mm:PinHeader_1x04_P2.54mm_Vertical
- J3: footprint Pin_Headers:Pin_Header_Straight_1x03_Pitch2.54mm -> Connector_PinHeader_2.54mm:PinHeader_1x03_P2.54mm_Vertical
- SW1, SW2, SW3, SW4, SW5, SW6, SW7, SW8: footprint Buttons_Switches_THT:SW_PUSH_6mm -> Button_Switch_THT:SW_PUSH_6mm
Other:
- board text added: "BasilFX 08/2018 V1.1.0"
