File: pcb/Universal-Taster/Taster.kicad_pcb (KiCad board)
At the start: 2 copper layers, 30 x 30 mm, 59 parts, among them J1 I2C, J2 INTERFACE, J3 KNX_KLEMME, J4 JTAG, SW1 PROG, U1 EFM32PG12B500, U2 NCN5121, U3 MX25R8035F, Y1 32.768kHz, Y2 40MHz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

Commit message: Upgrade Universal Taster to KiCad 6.0
Parts:
- J3: value KNX_KLEMME -> Val**
- L1: footprint PowerSwap:SRR5028 -> Inductors_SMD2:L_Bourns-SRR5028
- U3: footprint PowerSwap:winbond-USON-8(2X3UX) -> Package_USON:USON-8_2x3mm_P0.5mm
Connections:
- net 3V3-A renamed +3.3V
- J1 pad MP: (no net) -> GND
- J2 pad MP: (no net) -> GND
- U1 pad 13: Net-(U1-Pad13) -> unconnected-(U1-Pad13)
- U1 pad 14: Net-(U1-Pad14) -> unconnected-(U1-Pad14)
- U1 pad 15: Net-(U1-Pad15) -> unconnected-(U1-Pad15)
- U1 pad 16: Net-(U1-Pad16) -> unconnected-(U1-Pad16)
- U1 pad 17: Net-(U1-Pad17) -> unconnected-(U1-Pad17)
- U1 pad 18: Net-(U1-Pad18) -> unconnected-(U1-Pad18)
- U1 pad 19: Net-(U1-Pad19) -> unconnected-(U1-Pad19)
- U1 pad 20: Net-(U1-Pad20) -> unconnected-(U1-Pad20)
- U1 pad 27: Net-(U1-Pad27) -> unconnected-(U1-Pad27)
- U1 pad 28: Net-(U1-Pad28) -> unconnected-(U1-Pad28)
- U1 pad 29: Net-(U1-Pad29) -> unconnected-(U1-Pad29)
- U1 pad 30: Net-(U1-Pad30) -> unconnected-(U1-Pad30)
- U1 pad 31: Net-(U1-Pad31) -> unconnected-(U1-Pad31)
- U1 pad 38: Net-(U1-Pad38) -> unconnected-(U1-Pad38)
- U2 pad 12: Net-(U2-Pad12) -> unconnected-(U2-Pad12)
- U2 pad 13: Net-(U2-Pad13) -> unconnected-(U2-Pad13)
- U2 pad 15: Net-(U2-Pad15) -> unconnected-(U2-Pad15)
- U2 pad 21: Net-(U2-Pad21) -> unconnected-(U2-Pad21)
- U2 pad 22: Net-(U2-Pad22) -> unconnected-(U2-Pad22)
- U2 pad 32: Net-(U2-Pad32) -> unconnected-(U2-Pad32)
- U2 pad 39: Net-(U2-Pad39) -> unconnected-(U2-Pad39)
Routing:
- net GND: track 142.6 -> 99.3 mm
- net Net-(L1-Pad2): track 11.4 -> 9.59 mm
- net Net-(D2-Pad2): track 7.95 -> 6.40 mm
- net +3.3V: track 98.5 -> 97.2 mm
- net /KNX+: track 27.8 -> 26.7 mm
- net Net-(L1-Pad1): track 15.4 -> 14.2 mm
- net /RXD: track 7.91 -> 6.81 mm
- net /SWDCLK: track 4.60 -> 3.77 mm
- net /MISO: track 4.00 -> 3.30 mm
- net /SCL: track 14.6 -> 14.0 mm
- net Net-(D11-Pad1): track 4.55 -> 4.02 mm
- net /SWITCH: track 9.23 -> 9.75 mm
- net Net-(D6-Pad1): track 4.53 -> 4.02 mm
Other:
- net class Default removed
- net class KNX removed
- net class Power removed
- net class Power-3V3 removed
- board text added: "BasilFX 09/2022 V1.3.0"
- board text removed: "BasilFX 07/2021 V1.2.1"
