File: pcb/Universal-Taster/Universal-Taster.kicad_sch (KiCad schematic)
At the start: 59 parts, among them J1 I2C, J2 INTERFACE, J3 KNX_KLEMME, J4 JTAG, SW1 PROG, U1 EFM32PG12B500, U2 NCN5121, U3 MX25R8035F, Y1 32.768kHz, Y2 40MHz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

Commit message: Add interactive BoM to Universal Taster
Parts:
- C1, C2: Order Number (none) -> Farnell: 2821267
- C10, C13, C16, C18, C19, C8, C9: Order Number (none) -> Farnell: 1833843
- C11: Notes (none) -> 35 V; Order Number (none) -> DigiKey: 732-8511-1-ND
- C12: Notes (none) -> 35 V, 2 R ESR; Order Number (none) -> Farnell: 2346944
- C14: Notes (none) -> 50 V; Order Number (none) -> Farnell: 2346906
- C15: Notes (none) -> 50 V; Order Number (none) -> Farnell: 2524870
- C17: Notes (none) -> 6.3 V, 0.1 R ESR; Order Number (none) -> DigiKey: 445-9104-1-ND
- C3: Notes (none) -> 35 V; Order Number (none) -> DigiKey: 587-1437-1-ND
- C4, C5: Order Number (none) -> Farnell: 2627461
- C6, C7: Order Number (none) -> Farnell: 1414600
- D10, D11, D4, D5, D6, D7, D8, D9: Order Number (none) -> Farnell: 2368172
- D2: Order Number (none) -> DigiKey: 1SMA40CAT3GOSCT-ND
- D3: Order Number (none) -> DigiKey: SS16T3GOSCT-ND
- J3: footprint KNX_KLEMME -> KNX:KNX_KLEMME; Notes (none) -> Two pins needed.; Order Number (none) -> DigiKey:36-1425-2-ND
- J4: Notes (none) -> Contra is 1865334.; Order Number (none) -> Farnell: 2308512
- L1: Order Number (none) -> DigiKey: SRR5028-221YCT-ND
- R1, R4, R5, R6, R7, R8, R9: Order Number (none) -> DigiKey: MCT0603-680-CFCT-ND
- R10, R11, R12, R13: Order Number (none) -> DigiKey: 311-0.0GRCT-ND
- R2: Order Number (none) -> Farnell: 2426565
- R3: Order Number (none) -> Farnell: 2078888
- SW1: Order Number (none) -> DigiKey: SW1020CT-ND
- TP1, TP2, TP3, TP4: now left out of the parts list
- U1: Order Number (none) -> DigiKey: 336-3941-ND
- U2: Order Number (none) -> DigiKey: NCN5121MNTWGOSCT-ND
- U3: Order Number (none) -> DigiKey: 1092-1207-1-ND
- Y1: Order Number (none) -> DigiKey: XC2288CT-ND
- Y2: Order Number (none) -> DigiKey: 1253-1120-1-ND
- Y3: Order Number (none) -> DigiKey: 1253-1348-1-ND
