File: pcb/Extensions/DSMR-Connector/DSMR-Connector.kicad_sch (KiCad schematic)
At the start: 9 parts, among them J1 RJ12, J2 Conn_01x04, Q1 BC847, U1 FOD8012

Commit message: Add interactive BoM to DSMR Connector
Parts:
- C1, C2: Order Number (none) -> Farnell: 1833843
- J1: Order Number (none) -> Farnell: 2135977
- Q1: Notes (none) -> General purpose.; Order Number (none) -> Farnell: 2533307
- R1, R2, R3: Order Number (none) -> Farnell: 2447230
- U1: Order Number (none) -> DigiKey: FOD8012A-ND
Changed lines of the file:
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@@
+      (effects (font (size 1.27 1.27)) hide)
+    )
+    (property "Order Number" "Farnell: 2135977" (id 4) (at 49.53 58.42 0)
       (effects (font (size 1.27 1.27)) hide)
     )
@@
     (property "Datasheet" "" (id 3) (at 136.525 57.15 0)
       (effects (font (size 1.27 1.27)) (justify left) hide)
+    )
+    (property "Order Number" "DigiKey: FOD8012A-ND" (id 4) (at 137.16 57.15 0)
+      (effects (font (size 1.27 1.27)) hide)
     )
     (pin "1")
@@
       (effects (font (size 1.27 1.27)) hide)
     )
+    (property "Order Number" "Farnell: 1833843" (id 4) (at 109.22 60.96 0)
+      (effects (font (size 1.27 1.27)) hide)
+    )
     (pin "1")
     (pin "2")
@@
     )
     (property "Datasheet" "~" (id 3) (at 168.91 59.69 0)
+      (effects (font (size 1.27 1.27)) hide)
+    )
+    (property "Order Number" "Farnell: 1833843" (id 4) (at 168.91 59.69 0)
       (effects (font (size 1.27 1.27)) hide)
     )
@@
       (effects (font (size 1.27 1.27)) hide)
     )
+    (property "Order Number" "Farnell: 2447230" (id 4) (at 99.06 60.96 0)
+      (effects (font (size 1.27 1.27)) hide)
+    )
     (pin "1")
     (pin "2")
@@
       (effects (font (size 1.27 1.27)) (justify left) hide)
     )
+    (property "Notes" "General purpose." (id 4) (at 205.74 68.58 0)
+      (effects (font (size 1.27 1.27)) hide)
+    )
+    (property "Order Number" "Farnell: 2533307" (id 5) (at 205.74 68.58 0)
+      (effects (font (size 1.27 1.27)) hide)
+    )
     (pin "1")
     (pin "2")
@@
     )
     (property "Datasheet" "~" (id 3) (at 208.28 50.8 0)
+      (effects (font (size 1.27 1.27)) hide)
+    )
+    (property "Order Number" "Farnell: 2447230" (id 4) (at 208.28 50.8 0)
       (effects (font (size 1.27 1.27)) hide)
     )
@@
       (effects (font (size 1.27 1.27)) hide)
     )
+    (property "Order Number" "Farnell: 2447230" (id 4) (at 195.58 68.58 0)
+      (effects (font (size 1.27 1.27)) hide)
+    )
